File: schematic/picerino_sn76489AN.kicad_pcb (KiCad board)
At the start: 2 copper layers, 83.8 x 53.5 mm, 23 parts, among them CON1 PICERINO-EDGE, J1 Conn_01x02, J2 Conn_01x02, J3 Conn_01x02, U1 sn76489an, U2 74LS00, U3 LM386, Y1 3.579545Mhz

Commit message: updated schematics to kicad v6
Other:
- net class Default removed
